File: Greaseweazle F1 in a Gotek Case (USB-A)/Greaseweazle F1 Gotek (USB-A).sch (KiCad schematic (older format))
At the start: 14 parts, among them CN1 FLOPPY, J1 USB A, J2 Floppy Power, J3 Programming Port, U1 Blue Pill

Commit message: Added features
* Added Activity LED
* Added resistor pack
* Added Blue Pill footprint
Parts:
- added D2: LED, LED_THT:LED_D3.0mm, symbol Device:LED
- added R9: 1.5K, Resistor_SMD:R_0805_2012Metric, symbol Greaseweazle-F1-Gotek-(USB-A)-rescue:R-GW-rescue-Greaseweazle-F1-Gotek-rescue
- added RN1: R_Network04, Resistor_THT:R_Array_SIP5, symbol Device:R_Network04
- R1, R2, R3, R4, R5, R6: symbol Greaseweazle-F1-Gotek-rescue:R-GW-rescue -> Greaseweazle-F1-Gotek-(USB-A)-rescue:R-GW-rescue-Greaseweazle-F1-Gotek-rescue
- R7: renamed from R8; symbol Greaseweazle-F1-Gotek-rescue:R-GW-rescue -> Greaseweazle-F1-Gotek-(USB-A)-rescue:R-GW-rescue-Greaseweazle-F1-Gotek-rescue
- R8: renamed from R7; symbol Greaseweazle-F1-Gotek-rescue:R-GW-rescue -> Greaseweazle-F1-Gotek-(USB-A)-rescue:R-GW-rescue-Greaseweazle-F1-Gotek-rescue
- U1: footprint Package_DIP:DIP-40_W15.24mm -> Kicad-STM32-master:YAAJ_BluePill_1; symbol Greaseweazle-F1-Gotek-rescue:TAOBAO-FF-GW-rescue -> YAAJ_BluePill:YAAJ_BluePill
Connections:
- net labels added: _ACT
- wire segments 105 -> 119
Other:
- note added: "ACT LED"
- note added: "Optionl: Replaces R1 to R4"
- note added: "PWR LED"
- note added: "[Optional] R7 replaces R10 on the Blue Pill.\nYou MUST remove R10 on the Blue Pill\nwhen installing R7."
- moved on the sheet: D1, J1, J2, J3, R5, R6, R7, R8
