File: Greaseweazle F1 in a Gotek Case (USB-A)/Greaseweazle F1 Gotek (USB-A).sch (KiCad schematic (older format))
At the start: 18 parts, among them CN1 FLOPPY, J1 USB A, J2 Floppy Power, J3 Programming Port, SW1 SW_Push, U1 Blue Pill

Commit message: Tweaks and gerber files
Parts:
- CN1: value FLOPPY -> Floppy Data
- D1, D2: footprint Greaseweazle F1 in a Gotek Case (USB-A):LED_D3.0mm_Horizontal_O6.35mm_Z10.0mm_NoSilkS -> LED_THT:LED_D3.0mm_Horizontal_O6.35mm_Z10.0mm
- SW1: value SW_Push -> Reset
Changed lines of the file:
@@
 P 10650 5250
 F 0 "CN1" H 10650 6150 50  0000 C CNN
-F 1 "FLOPPY" V 10650 5250 50  0000 C CNN
+F 1 "Floppy Data" V 10650 5250 50  0000 C CNN
 F 2 "Connector_PinHeader_2.54mm:PinHeader_2x17_P2.54mm_Vertical" H 10650 4150 60  0001 C CNN
 F 3 "" H 10650 4150 60  0000 C CNN
@@
 F 0 "D1" H 8843 2216 50  0000 C CNN
 F 1 "LED" H 8843 2125 50  0000 C CNN
-F 2 "Greaseweazle F1 in a Gotek Case (USB-A):LED_D3.0mm_Horizontal_O6.35mm_Z10.0mm_NoSilkS" H 8850 2000 50  0001 C CNN
+F 2 "LED_THT:LED_D3.0mm_Horizontal_O6.35mm_Z10.0mm" H 8850 2000 50  0001 C CNN
 F 3 "~" H 8850 2000 50  0001 C CNN
 	1    8850 2000
@@
 F 0 "D2" H 9943 2216 50  0000 C CNN
 F 1 "LED" H 9943 2125 50  0000 C CNN
-F 2 "Greaseweazle F1 in a Gotek Case (USB-A):LED_D3.0mm_Horizontal_O6.35mm_Z10.0mm_NoSilkS" H 9950 2000 50  0001 C CNN
+F 2 "LED_THT:LED_D3.0mm_Horizontal_O6.35mm_Z10.0mm" H 9950 2000 50  0001 C CNN
 F 3 "~" H 9950 2000 50  0001 C CNN
 	1    9950 2000
@@
 P 5900 4650
 F 0 "SW1" H 5900 4935 50  0000 C CNN
-F 1 "SW_Push" H 5900 4844 50  0000 C CNN
+F 1 "Reset" H 5900 4844 50  0000 C CNN
 F 2 "OpenFlops:PUSH_BUTTON_RIGHT_ANGLE" H 5900 4850 50  0001 C CNN
 F 3 "~" H 5900 4850 50  0001 C CNN
