File: Greaseweazle F1 in a Gotek Case (USB-A)/Greaseweazle F1 Gotek (USB-A).sch (KiCad schematic (older format))
At the start: 18 parts, among them CN1 Floppy Data, J1 USB A, J2 Floppy Power, J3 Programming Port, SW1 Reset, U1 Blue Pill

Commit message: Tweaks after first build test
* Increased size of silk screen text
* Moved notch down a bit
* Swap +5V and GND on Programming port
* Moved LED holes nearer towards front.
Changed lines of the file:
@@
 L power:GND #PWR0115
 U 1 1 5FDBDC26
-P 6050 3100
-F 0 "#PWR0115" H 6050 2850 50  0001 C CNN
-F 1 "GND" H 6050 2950 50  0000 C CNN
-F 2 "" H 6050 3100 60  0000 C CNN
-F 3 "" H 6050 3100 60  0000 C CNN
-	1    6050 3100
+P 6400 3100
+F 0 "#PWR0115" H 6400 2850 50  0001 C CNN
+F 1 "GND" H 6400 2950 50  0000 C CNN
+F 2 "" H 6400 3100 60  0000 C CNN
+F 3 "" H 6400 3100 60  0000 C CNN
+	1    6400 3100
 	1    0    0    -1
 $EndComp
 Wire Wire Line
-	6750 2750 6050 2750
-Wire Wire Line
-	6050 2750 6050 2450
-Wire Wire Line
 	6750 2850 6050 2850
 Wire Wire Line
-	6050 2850 6050 3100
+	6050 2850 6050 2450
+Wire Wire Line
+	6750 2750 6400 2750
+Wire Wire Line
+	6400 2750 6400 3100
 Text Label 6300 2650 0    60   ~ 0
 SER_TX
