File: Greaseweazle F1 3.5 Inch/Greaseweazle F1 3.5 Inch.sch (KiCad schematic (older format))
At the start: 33 parts, among them CN1 Floppy Data, J1 USB B, J10 Conn_01x03, J11 Conn_01x03, J2 USB Header, J3 Floppy Power, J4 Floppy Power Header, J5 Programming Port, J6 SWD Port, J7 SWD Port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

Commit message: Added 12V LED
Parts:
- gave numbers to parts that had none: 2
Changed lines of the file:
@@
 	6575 4600 6575 4675
 $Comp
-L Device:LED D?
+L Device:LED D4
 U 1 1 5FDFF47A
 P 10300 2050
-F 0 "D?" H 10293 2266 50  0000 C CNN
+F 0 "D4" H 10293 2266 50  0000 C CNN
 F 1 "+5V LED" H 10293 2175 50  0000 C CNN
 F 2 "LED_SMD:LED_0805_2012Metric_Pad1.15x1.40mm_HandSolder" H 10300 2050 50  0001 C CNN
@@
 	10150 2050 9950 2050
 $Comp
-L Device:R R?
+L Device:R R11
 U 1 1 5FDFF486
 P 10750 2050
-F 0 "R?" V 10830 2050 50  0000 C CNN
+F 0 "R11" V 10830 2050 50  0000 C CNN
 F 1 "4.7K" V 10750 2050 50  0000 C CNN
 F 2 "Resistor_SMD:R_0805_2012Metric_Pad1.15x1.40mm_HandSolder" V 10680 2050 30  0001 C CNN
@@
 	9950 2050 9950 2300
 $Comp
-L power:GND #PWR?
+L power:GND #PWR0135
 U 1 1 5FDFF492
 P 9950 2300
-F 0 "#PWR?" H 9950 2050 50  0001 C CNN
+F 0 "#PWR0135" H 9950 2050 50  0001 C CNN
 F 1 "GND" H 9950 2150 50  0000 C CNN
 F 2 "" H 9950 2300 60  0000 C CNN
@@
 $EndComp
 $Comp
-L power:+12V #PWR?
+L power:+12V #PWR0136
 U 1 1 5FE199DC
 P 10900 1800
-F 0 "#PWR?" H 10900 1650 50  0001 C CNN
+F 0 "#PWR0136" H 10900 1650 50  0001 C CNN
 F 1 "+12V" H 10915 1973 50  0000 C CNN
 F 2 "" H 10900 1800 50  0001 C CNN
