File: Greaseweazle F1 Gotek Rev 2/Greaseweazle F1 Gotek Rev 2.sch (KiCad schematic (older format))
At the start: 34 parts, among them CN1 Floppy Data, J1 SWD, J2 Floppy Power, J3 Programming Port, J4 USB B, J5 Boot Header, J6 LEDC68, P1 12V Power, SW1 Reset, U1 Blue Pill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

Commit message: Corrected 12V LED resistor from 2K to 4.7K
Parts:
- R11: value 2K -> 4.7K
Connections:
- no-connect marks 21 -> 24
Other:
- moved on the sheet: C1, C2, P1, U2
Changed lines of the file:
@@
 L Connector:Conn_01x03_Male P1
 U 1 1 601D6AEC
-P 1675 975
-F 0 "P1" H 1325 1250 50  0000 L CNN
-F 1 "12V Power" H 1325 1150 50  0000 L CNN
-F 2 "Connector_BarrelJack:BarrelJack_Horizontal" H 1675 975 50  0001 C CNN
-F 3 "~" H 1675 975 50  0001 C CNN
-	1    1675 975
+P 950 1025
+F 0 "P1" H 600 1300 50  0000 L CNN
+F 1 "12V Power" H 600 1200 50  0000 L CNN
+F 2 "Connector_BarrelJack:BarrelJack_Horizontal" H 950 1025 50  0001 C CNN
+F 3 "~" H 950 1025 50  0001 C CNN
+	1    950  1025
 	1    0    0    -1
 $EndComp
@@
 L power:+12V #PWR0110
 U 1 1 601EDAE7
-P 2050 750
-F 0 "#PWR0110" H 2050 600 50  0001 C CNN
-F 1 "+12V" H 2065 923 50  0000 C CNN
-F 2 "" H 2050 750 50  0001 C CNN
-F 3 "" H 2050 750 50  0001 C CNN
-	1    2050 750
-	1    0    0    -1
-$EndComp
-Wire Wire Line
-	2050 750  2050 775
-Wire Wire Line
-	2050 875  1875 875
+P 1325 800
+F 0 "#PWR0110" H 1325 650 50  0001 C CNN
+F 1 "+12V" H 1340 973 50  0000 C CNN
+F 2 "" H 1325 800 50  0001 C CNN
+F 3 "" H 1325 800 50  0001 C CNN
+	1    1325 800
+	1    0    0    -1
+$EndComp
+Wire Wire Line
+	1325 800  1325 825
+Wire Wire Line
+	1325 925  1150 925
 $Comp
 L power:PWR_FLAG #FLG0104
 U 1 1 601F5417
-P 2050 775
-F 0 "#FLG0104" H 2050 850 50  0001 C CNN
-F 1 "PWR_FLAG" V 2050 903 50  0000 L CNN
-F 2 "" H 2050 775 50  0001 C CNN
-F 3 "~" H 2050 775 50  0001 C CNN
-	1    2050 775
+P 1325 825
+F 0 "#FLG0104" H 1325 900 50  0001 C CNN
+F 1 "PWR_FLAG" V 1325 953 50  0000 L CNN
+F 2 "" H 1325 825 50  0001 C CNN
+F 3 "~" H 1325 825 50  0001 C CNN
+	1    1325 825
 	0    1    1    0
 $EndComp
-Connection ~ 2050 775
-Wire Wire Line
-	2050 775  2050 875
+Connection ~ 1325 825
+Wire Wire Line
+	1325 825  1325 925
 $Comp
 L power:GND #PWR0126
 U 1 1 601FC944
-P 2050 1150
-F 0 "#PWR0126" H 2050 900 50  0001 C CNN
-F 1 "GND" H 2050 1000 50  0000 C CNN
-F 2 "" H 2050 1150 60  0000 C CNN
-F 3 "" H 2050 1150 60  0000 C CNN
-	1    2050 1150
-	1    0    0    -1
-$EndComp
-Wire Wire Line
-	1875 975  2050 975
-Wire Wire Line
-	1875 1075 2050 1075
-Wire Wire Line
-	2050 975  2050 1075
-Connection ~ 2050 1075
-Wire Wire Line
-	2050 1075 2050 1150
+P 1325 1200
+F 0 "#PWR0126" H 1325 950 50  0001 C CNN
+F 1 "GND" H 1325 1050 50  0000 C CNN
+F 2 "" H 1325 1200 60  0000 C CNN
+F 3 "" H 1325 1200 60  0000 C CNN
+	1    1325 1200
+	1    0    0    -1
+$EndComp
+Wire Wire Line
+	1150 1025 1325 1025
+Wire Wire Line
+	1150 1125 1325 1125
+Wire Wire Line
+	1325 1025 1325 1125
+Connection ~ 1325 1125
+Wire Wire Line
+	1325 1125 1325 1200
 $Comp
 L power:+12V #PWR0127
@@
 P 10525 950
 F 0 "R11" V 10605 950 50  0000 C CNN
-F 1 "2K" V 10525 950 50  0000 C CNN
+F 1 "4.7K" V 10525 950 50  0000 C CNN
 F 2 "Resistor_SMD:R_0805_2012Metric" V 10455 950 30  0001 C CNN
 F 3 "" H 10525 950 30  0000 C CNN
@@
 L Regulator_Linear:AP2112K-3.3 U2
 U 1 1 5FE635B1
-P 4150 1225
-F 0 "U2" H 4150 1567 50  0000 C CNN
-F 1 "AP2112K-3.3" H 4150 1476 50  0000 C CNN
-F 2 "Package_TO_SOT_SMD:SOT-23-5" H 4150 1550 50  0001 C CNN
-F 3 "https://www.diodes.com/assets/Datasheets/AP2112.pdf" H 4150 1325 50  0001 C CNN
-	1    4150 1225
+P 4075 1100
+F 0 "U2" H 4075 1442 50  0000 C CNN
+F 1 "AP2112K-3.3" H 4075 1351 50  0000 C CNN
+F 2 "Package_TO_SOT_SMD:SOT-23-5" H 4075 1425 50  0001 C CNN
+F 3 "https://www.diodes.com/assets/Datasheets/AP2112.pdf" H 4075 1200 50  0001 C CNN
+	1    4075 1100
 	1    0    0    -1
 $EndComp
@@
 L Device:C C1
 U 1 1 5FE648E8
-P 3425 1375
-F 0 "C1" H 3540 1421 50  0000 L CNN
-F 1 "1u" H 3540 1330 50  0000 L CNN
-F 2 "Capacitor_SMD:C_0805_2012Metric_Pad1.15x1.40mm_HandSolder" H 3463 1225 50  0001 C CNN
-F 3 "~" H 3425 1375 50  0001 C CNN
-	1    3425 1375
+P 3350 1250
+F 0 "C1" H 3465 1296 50  0000 L CNN
+F 1 "1u" H 3465 1205 50  0000 L CNN
+F 2 "Capacitor_SMD:C_0805_2012Metric_Pad1.15x1.40mm_HandSolder" H 3388 1100 50  0001 C CNN
+F 3 "~" H 3350 1250 50  0001 C CNN
+	1    3350 1250
 	1    0    0    -1
 $EndComp
@@
 L Device:C C2
 U 1 1 5FE657CF
-P 4750 1375
-F 0 "C2" H 4865 1421 50  0000 L CNN
-F 1 "1u" H 4865 1330 50  0000 L CNN
-F 2 "Capacitor_SMD:C_0805_2012Metric_Pad1.15x1.40mm_HandSolder" H 4788 1225 50  0001 C CNN
-F 3 "~" H 4750 1375 50  0001 C CNN
-	1    4750 1375
+P 4675 1250
+F 0 "C2" H 4790 1296 50  0000 L CNN
+F 1 "1u" H 4790 1205 50  0000 L CNN
+F 2 "Capacitor_SMD:C_0805_2012Metric_Pad1.15x1.40mm_HandSolder" H 4713 1100 50  0001 C CNN
+F 3 "~" H 4675 1250 50  0001 C CNN
+	1    4675 1250
 	1    0    0    -1
 $EndComp
@@
 L power:GND #PWR0132
 U 1 1 5FE65D74
-P 4150 1650
-F 0 "#PWR0132" H 4150 1400 50  0001 C CNN
-F 1 "GND" H 4150 1500 50  0000 C CNN
-F 2 "" H 4150 1650 60  0000 C CNN
-F 3 "" H 4150 1650 60  0000 C CNN
-	1    4150 1650
-	1    0    0    -1
-$EndComp
-Wire Wire Line
-	4150 1525 4150 1650
-Wire Wire Line
-	3425 1525 4150 1525
-Connection ~ 4150 1525
-Wire Wire Line
-	4150 1525 4750 1525
+P 4075 1525
+F 0 "#PWR0132" H 4075 1275 50  0001 C CNN
+F 1 "GND" H 4075 1375 50  0000 C CNN
+F 2 "" H 4075 1525 60  0000 C CNN
+F 3 "" H 4075 1525 60  0000 C CNN
+	1    4075 1525
+	1    0    0    -1
+$EndComp
+Wire Wire Line
+	4075 1400 4075 1525
+Wire Wire Line
+	3350 1400 4075 1400
+Connection ~ 4075 1400
+Wire Wire Line
+	4075 1400 4675 1400
 $Comp
 L power:+5V #PWR0133
 U 1 1 5FE7EE0F
-P 3425 950
-F 0 "#PWR0133" H 3425 800 50  0001 C CNN
-F 1 "+5V" H 3425 1090 50  0000 C CNN
-F 2 "" H 3425 950 60  0000 C CNN
-F 3 "" H 3425 950 60  0000 C CNN
-	1    3425 950
-	1    0    0    -1
-$EndComp
-Wire Wire Line
-	3850 1125 3725 1125
-Wire Wire Line
-	3425 1125 3425 950
-Wire Wire Line
-	3425 1225 3425 1125
-Connection ~ 3425 1125
-Wire Wire Line
-	4450 1125 4750 1125
-Wire Wire Line
-	4750 1125 4750 1025
-Wire Wire Line
-	4750 1125 4750 1225
-Connection ~ 4750 1125
+P 3350 825
+F 0 "#PWR0133" H 3350 675 50  0001 C CNN
+F 1 "+5V" H 3350 965 50  0000 C CNN
+F 2 "" H 3350 825 60  0000 C CNN
+F 3 "" H 3350 825 60  0000 C CNN
+	1    3350 825
+	1    0    0    -1
+$EndComp
+Wire Wire Line
+	3775 1000 3650 1000
+Wire Wire Line
+	3350 1000 3350 825
+Wire Wire Line
+	3350 1100 3350 1000
+Connection ~ 3350 1000
+Wire Wire Line
+	4375 1000 4675 1000
+Wire Wire Line
+	4675 1000 4675 900
+Wire Wire Line
+	4675 1000 4675 1100
+Connection ~ 4675 1000
 $Comp
 L power:PWR_FLAG #FLG0105
 U 1 1 5FEBD53D
-P 4750 1025
-F 0 "#FLG0105" H 4750 1100 50  0001 C CNN
-F 1 "PWR_FLAG" V 4750 1153 50  0000 L CNN
-F 2 "" H 4750 1025 50  0001 C CNN
-F 3 "~" H 4750 1025 50  0001 C CNN
-	1    4750 1025
+P 4675 900
+F 0 "#FLG0105" H 4675 975 50  0001 C CNN
+F 1 "PWR_FLAG" V 4675 1028 50  0000 L CNN
+F 2 "" H 4675 900 50  0001 C CNN
+F 3 "~" H 4675 900 50  0001 C CNN
+	1    4675 900
 	0    1    1    0
 $EndComp
-Connection ~ 4750 1025
-Wire Wire Line
-	4750 1025 4750 875
+Connection ~ 4675 900
+Wire Wire Line
+	4675 900  4675 750
 Connection ~ 3550 4250
 $Comp
@@
 	0    1    1    0
 $EndComp
-Text Label 4750 875  0    50   ~ 0
+Text Label 4675 750  0    50   ~ 0
 USB_3V3
 Wire Wire Line
-	3850 1225 3725 1225
-Wire Wire Line
-	3725 1225 3725 1125
-Connection ~ 3725 1125
-Wire Wire Line
-	3725 1125 3425 1125
+	3775 1100 3650 1100
+Wire Wire Line
+	3650 1100 3650 1000
+Connection ~ 3650 1000
+Wire Wire Line
+	3650 1000 3350 1000
 $Comp
 L MCU_Module:Arduino_Nano_v3.x A1
@@
 Text Label 5975 5700 0    60   ~ 0
 _RST
+NoConn ~ 6950 4600
+NoConn ~ 6975 5250
+NoConn ~ 6975 5900
 $EndSCHEMATC
