File: Greaseweazle F1 Gotek Rev 2/_autosave-Greaseweazle F1 Gotek Rev 2.kicad_pcb (KiCad board)
At the start: 2 copper layers, 111.6 x 94.4 mm, 56 parts, among them CN1 Floppy Data, J1 PinHeader_1x04_P2.54mm_Vertic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, J1 SWD, J2 Floppy Power, J2 PinHeader_1x04_P2.54mm_Vertic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, J3 PinHeader_1x04_P2.54mm_Vertic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, J3 Programming Port, J4 USB B, J5 Boot Header, J6 LEDC68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

Commit message: Added DWGS.User layer
Parts:
- added REF**: Floppy_Drive, solarmon_library:Floppy_Drive, F.Cu at (154.2, 85.9)
