File: Blue Pill Kickstart Switcher/Blue Pill Kickstart Switcher.kicad_pcb (KiCad board)
At the start: 2 copper layers, 65.4 x 76.8 mm, 23 parts, among them J1 Conn_01x02, J2 Conn_01x03, J3 Conn_01x03, J4 Conn_01x04, J5 Conn_01x03, J6 Conn_01x02, J7 Conn_01x02, J8 Conn_01x02, J9 Conn_01x02, U1 Conn_02x21_Counter_Clockwise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

Commit message: Show resistor values in silk screen
Parts:
- R1, R2, R3, R4: value R -> 4K7
Other:
- board text added: "* Hold down reset (CTRL-A-A) to cycle through ROM slots. Buzzer will sound for each transition. * Use Serial Config to program ROM slots. * Enable Serial Config with J7 (and disconnect other jumpers)"
- board text removed: "* Hold down reset (CTRL-A-A) to cycle through ROM slots. Buzzer will sound for each transition. * Use Serial Config to program ROM slots. * Enable Serial Config with J7"
